File: PCB/prototypeBoard/nrf52withamp.brd (EAGLE design)
At the start: 160 x 100 mm, 90 parts, among them Q3 DMG3415U-7, SW1 KMR2, SW2 KMR2, U1 MDBT42, U2 AP2112(3.3V), U3 MCP73831T-2ACI/OT, U4 LMV324, U5 AP2112(3.3V), U6 PAM8302AASCR, U7 PAM8302AASCR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

Commit message: update code
Parts:
- removed TP3, TP4: (no value), microbuilder:TESTPOINT_ROUND_2MM
- added J5, J6: (no value), SparkFun-Connectors:1X04_1.27MM
- added JP4: SWO, microbuilder:1X01_2MM
- SW1: value KMR2 -> RST
- SW2: value KMR2 -> DFU
- moved C15 212.6 mm to (25.7, 63.5)
- moved R17 210.8 mm to (27.9, 59.7), turned to 270 degrees
- moved U5 205.4 mm to (24.9, 59.7), turned to 180 degrees
- moved C16 198.6 mm to (25.7, 55.9), turned to 180 degrees
- moved C8 183.6 mm to (27.4, 71.6), turned to 90 degrees
- moved U2 182.9 mm to (31.5, 71.6), turned to 90 degrees
- moved R11 174.2 mm to (3.05, 63.8), turned to 90 degrees
- moved C6 173.8 mm to (35.6, 71.6), turned to 90 degrees
- moved R6 172.4 mm to (30.7, 79.8)
- moved R14 172.4 mm to (5.59, 69.1), turned to 90 degrees
- moved C9 171.3 mm to (23.4, 78.5)
- moved C12 170.5 mm to (30.7, 82.8)
- moved Q3 170.5 mm to (38.6, 68.3), turned to 180 degrees
- moved C7 170.4 mm to (21.1, 78.5)
- moved J1 170.1 mm to (37.1, 94.7)
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Connections:
- net A7/P0.31 renamed A7/0.31
- net N$13 renamed AMP_REF
- removed net A6/P0.30: U1.7
- new net A6/0.30: J6.2, U1.7
- new net EN_VCC2: R17.2, U5.3
- net 3.3V: now also J6.1
- net A4/0.28: now also J6.4
- net A5/0.29: now also J6.3
- net EN: no longer R17.2, U5.3
- net GND: now also J5.1
- net P0.27: now also J5.4
- net SCL: now also J5.3
- net SDA: now also J5.2
- net SWCLK: no longer TP4.P$1
- net SWDIO: no longer TP3.P$1
- net SWO: now also JP4.1
Routing:
- net GND: track 0.00 -> 225.1 mm, vias 0 -> 13
- net 3.3V: track 0.00 -> 76.8 mm, vias 0 -> 5
- net VBAT: track 0.00 -> 38.0 mm, vias 0 -> 2
- net A7/0.31: track 0.00 -> 36.5 mm, vias 0 -> 2
- net VIN: track 0.00 -> 31.9 mm
- net VBUS: track 0.00 -> 24.8 mm, vias 0 -> 2
- net RESET: track 0.00 -> 23.5 mm
- net SWCLK: track 0.00 -> 19.2 mm
- net LED2: track 0.00 -> 17.2 mm, vias 0 -> 2
- net DFU: track 0.00 -> 15.3 mm
- net A0/0.02: track 0.00 -> 12.1 mm
- net SWDIO: track 0.00 -> 11.9 mm
- net LED1: track 0.00 -> 11.8 mm, vias 0 -> 2
- net N$6: track 0.00 -> 10.1 mm
- net N$9: track 0.00 -> 9.96 mm
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Other:
- board size 160 x 100 mm -> 44.5 x 101.6 mm

Commit message: add PCB
Parts:
- removed C24, C25: 1uF, microbuilder:0805-NO
- removed C26: 10uF, microbuilder:0805-NO
- removed C27, C28: 220pF, microbuilder:0805-NO
- removed FB3, FB4: Ferrite, microbuilder:_0805
- removed R23, R24: 100, microbuilder:0805-NO
- removed R25: 10K, microbuilder:0805-NO
- removed R26, R27: 5K, rcl:R0805
- removed U7: PAM8302AASCR, microbuilder:MSOP8_0.65MM
- added C29: 100nF, rcl:C0805
- added C30, C37: TBD, microbuilder:0805-NO
- added C32, C33: 1uF, microbuilder:0805-NO
- added C34: 10uF, microbuilder:0805-NO
- added C35, C36: 220pF, microbuilder:0805-NO
- added D4: 1N4148, microbuilder:SOD-323
- added FB5, FB6: Ferrite, microbuilder:_0805
- added J10, J11, J12, J13, J14, J15: (no value), SparkFun-Connectors:1X07
- added J7: (no value), SparkFun-Connectors:6_PIN_SERIAL_TARGET_SIDE_RA_SMT
- added J8: (no value), SparkFun-Connectors:1X04_1.27MM
- added J9: (no value), SparkFun-Connectors:1X02
- added R28: 10k, rcl:R0805
- added R29, R30: 1k, rcl:R0805
- added R31, R32: 100, microbuilder:0805-NO
- added R33: 10K, microbuilder:0805-NO
- added R34, R35: 5K, rcl:R0805
- added SJ2: BAT, microbuilder:SOLDERJUMPER_CLOSEDWIRE
- added U8: PAM8302AASCR, microbuilder:MSOP8_0.65MM
- J4: device SparkFun-Connectors:1X02 -> SparkFun-Connectors:1X07
- moved R22 307.7 mm to (19.3, 21.1), turned to 270 degrees
- moved J4 298.1 mm to (26.7, 41.9)
- moved C19 259.5 mm to (21.8, 21.1), turned to 270 degrees
- moved R19 257.7 mm to (24.4, 21.1), turned to 270 degrees
- moved R21 256.3 mm to (19.3, 16.8), turned to 270 degrees
- moved U6 253.3 mm to (29.5, 21.1)
- moved C20 251.8 mm to (21.8, 16.8), turned to 90 degrees
- moved R18 250.0 mm to (24.4, 16.8), turned to 90 degrees
- moved FB2 248.0 mm to (35.3, 21.6)
- moved FB1 247.8 mm to (35.3, 15.0)
- moved C22 247.2 mm to (38.9, 20.6)
- moved C21 245.5 mm to (34.3, 18.3), turned to 90 degrees
- moved R20 245.5 mm to (29.5, 18.0)
- moved C23 244.7 mm to (38.9, 15.7)
- moved J3 242.2 mm to (41.7, 15.5)
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Connections:
- removed net N$26: R23.2, U7.4
- removed net N$27: R24.2, U7.3
- removed net N$28: C25.1, R23.1
- removed net N$29: FB4.1, U7.8
- removed net N$30: FB3.1, U7.5
- removed net N$31: C24.1, R24.1
- removed net N$32: C24.2, R26.1, R27.2
- removed net SD: R20.2, R25.2, U6.1, U7.1
- removed net VO+: C23.1, C28.1, FB1.2, FB3.2, J3.1, J4.1
- removed net VO-: C22.1, C27.1, FB2.2, FB4.2, J3.2, J4.2
- new net DTR: C29.1, J7.1
- new net N$13: C29.2, SJ2.2
- new net N$33: J7.3, R29.1
- new net N$34: J7.2, R30.1
- new net N$35: R31.2, U8.4
- new net N$36: R32.2, U8.3
- new net N$37: C33.1, R31.1
- new net N$38: FB6.1, U8.8
- new net N$39: FB5.1, U8.5
- new net N$40: C32.1, R32.1
- new net N$41: C32.2, C37.1, R34.1, R35.2
- new net SD1: R20.2, U6.1
- new net SD2: R33.2, U8.1
- new net VO1+: C23.1, FB1.2, J3.1
- new net VO1-: C22.1, FB2.2, J3.2
- new net VO2+: C36.1, FB5.2, J9.1
- new net VO2-: C35.1, FB6.2, J9.2
- net 3.3V: now also D4.C, R28.1
- net A1/0.03: now also J8.1
- net A2/0.04: now also J8.2
- net A3/0.05: now also J8.3
- net GND: now also C34.2, C35.2, C36.2, J7.6, J8.4, U8.7; no longer C26.2, C27.2, C28.2, U7.7
- net N$25: now also C30.1
- net P0.07: now also C30.2
- net P0.15: now also R35.1; no longer R27.1
- net P0.16: now also C33.2, C37.2, R34.2; no longer C25.2, R26.2
- net RESET: now also D4.A, R28.2, SJ2.1
- net RXD: now also R30.2
- net TXD: now also R29.2
- net VBUS: now also J7.4
- net VCC_2: now also C34.1, R33.1, U8.6; no longer C26.1, R25.1, U7.6
Routing:
- net GND: track 225.1 -> 482.5 mm, vias 13 -> 19
- net VCC_2: track 2.83 -> 137.9 mm, vias 0 -> 7
- net P0.16: track 0.00 -> 104.4 mm, vias 0 -> 4
- net P0.15: track 0.00 -> 86.4 mm, vias 0 -> 4
- net MOSI: track 0.00 -> 78.5 mm, vias 0 -> 2
- net SCK: track 0.00 -> 77.8 mm, vias 0 -> 2
- net RESET: track 23.5 -> 97.1 mm, vias 0 -> 2
- net P0.07: track 0.00 -> 72.7 mm, vias 0 -> 2
- net 3.3V: track 76.8 -> 139.9 mm, vias 5 -> 7
- net P0.11: track 0.00 -> 62.9 mm, vias 0 -> 2
- net TXD: track 0.00 -> 47.3 mm, vias 0 -> 2
- net RXD: track 0.00 -> 45.5 mm, vias 0 -> 2
- net VBUS: track 24.8 -> 64.3 mm, vias 2 -> 4
- net AMP_REF: track 9.36 -> 38.5 mm, vias 0 -> 4
- net VCCA: track 3.39 -> 21.9 mm, vias 0 -> 2
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Other:
- board size 44.5 x 101.6 mm -> 44.5 x 94 mm

Commit message: update board
Parts:
- removed C32, C33: 1uF, microbuilder:0805-NO
- removed C34: 10uF, microbuilder:0805-NO
- removed R33: 10K, microbuilder:0805-NO
- added C24, C26: 1uF, rcl:C0805
- added C25: 10uF, rcl:C0805
- added R24: 10k, rcl:R0805
- added SW3: SWITCH_SPDT, SparkFun-Retired:KPS-1290
- C19, C20, C21: device microbuilder:0805-NO -> rcl:C0805
- JP4: value SWO -> (none)
- R20: value 10K -> 10k; device microbuilder:0805-NO -> rcl:R0805
- moved C21 1.02 mm to (35.3, 18.3), turned to 0 degrees
- moved R20 0.25 mm to (29.5, 18.3), turned to 0 degrees
- turned C19 to 90 degrees
- turned C20 to 270 degrees
Connections:
- new net N$26: Q3.3, SW3.S
- net GND: now also C25.2; no longer C34.2
- net N$21: now also C20.2; no longer C20.1
- net N$24: now also C19.2; no longer C19.1
- net N$25: now also C19.1; no longer C19.2
- net N$37: now also C26.2; no longer C33.1
- net N$40: now also C24.2; no longer C32.1
- net N$41: now also C24.1; no longer C32.2
- net P0.07: now also C20.1; no longer C20.2
- net P0.16: now also C26.1; no longer C33.2
- net SD1: now also R20.1; no longer R20.2
- net SD2: now also R24.1; no longer R33.2
- net VBAT: now also SW3.P; no longer Q3.3
- net VCC_2: now also C25.1, R20.2, R24.2; no longer C34.1, R20.1, R33.1
Routing:
- net N$26: track 0.00 -> 46.8 mm, vias 0 -> 4
- net VBAT: track 38.0 -> 78.0 mm, vias 2 -> 6
- net GND: track 482.5 -> 488.0 mm, vias 19 -> 20
- net VCC_2: track 137.9 -> 143.4 mm, vias 7 -> 9
- net 3.3V: track 139.9 -> 141.9 mm
- net RESET: track 97.1 -> 98.1 mm
- net VIN: track 32.0 -> 31.0 mm
- net A0/0.02: track 12.1 -> 12.7 mm
- added copper zone on layer 16, net GND
Other:
- board text added: "ON"
- board text added: "SWO"
