File: PCB/prototypeBoard/nrf52withamp.sch (EAGLE design)
At the start: 90 parts, among them Q3 DMG3415U-7, SW1 KMR2, SW2 KMR2, U1 MDBT42, U2 AP2112(3.3V), U3 MCP73831T-2ACI/OT, U4 LMV324, U5 AP2112(3.3V), U6 PAM8302AASCR, U7 PAM8302AASCR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

Commit message: update code
Parts:
- removed TP3, TP4: (no value), microbuilder:TESTPOINTROUND2MM
- added J5, J6: (no value), SparkFun-Connectors:CONN_041.27MM
- added JP4: SWO, microbuilder:HEADER-1X12MM
- SW1: value KMR2 -> RST
- SW2: value KMR2 -> DFU
Connections:
- net A7/P0.31 renamed A7/0.31
- net N$13 renamed AMP_REF
- removed net A6/P0.30: U1.P0.30/AIN6
- new net A6/0.30: J6.2, U1.P0.30/AIN6
- new net EN_VCC2: R17.2, U5.EN
- net 3.3V: now also J6.1
- net A4/0.28: now also J6.4
- net A5/0.29: now also J6.3
- net EN: no longer R17.2, U5.EN
- net GND: now also J5.1
- net P0.27: now also J5.4
- net SCL: now also J5.3
- net SDA: now also J5.2
- net SWCLK: no longer TP4.P$1
- net SWDIO: no longer TP3.P$1
- net SWO: now also JP4.1
Other:
- moved on the sheet: R22

Commit message: add PCB
Parts:
- removed C24, C25: 1uF, microbuilder:CAP_CERAMIC0805-NOOUTLINE
- removed C26: 10uF, microbuilder:CAP_CERAMIC0805-NOOUTLINE
- removed C27, C28: 220pF, microbuilder:CAP_CERAMIC0805-NOOUTLINE
- removed FB3, FB4: Ferrite, microbuilder:FERRITE_0805
- removed R23, R24: 100, microbuilder:RESISTOR0805_NOOUTLINE
- removed R25: 10K, microbuilder:RESISTOR0805_NOOUTLINE
- removed R26, R27: 5K, rcl:R-EU_R0805
- removed U7: PAM8302AASCR, microbuilder:AUDIOAMP_PAM8302A
- added C29: 100nF, rcl:C-EUC0805
- added C30, C37: TBD, microbuilder:CAP_CERAMIC0805-NOOUTLINE
- added C32, C33: 1uF, microbuilder:CAP_CERAMIC0805-NOOUTLINE
- added C34: 10uF, microbuilder:CAP_CERAMIC0805-NOOUTLINE
- added C35, C36: 220pF, microbuilder:CAP_CERAMIC0805-NOOUTLINE
- added D4: 1N4148, microbuilder:DIODESOD-323
- added FB5, FB6: Ferrite, microbuilder:FERRITE_0805
- added J10, J11, J12, J13, J14, J15: (no value), SparkFun-Connectors:CONN_07
- added J7: (no value), SparkFun-Connectors:6_PIN_SERIAL_TARGETRA_SMT
- added J8: (no value), SparkFun-Connectors:CONN_041.27MM
- added J9: (no value), SparkFun-Connectors:CONN_02
- added R28: 10k, rcl:R-EU_R0805
- added R29, R30: 1k, rcl:R-EU_R0805
- added R31, R32: 100, microbuilder:RESISTOR0805_NOOUTLINE
- added R33: 10K, microbuilder:RESISTOR0805_NOOUTLINE
- added R34, R35: 5K, rcl:R-EU_R0805
- added SJ2: BAT, microbuilder:SOLDERJUMPERCLOSED
- added U8: PAM8302AASCR, microbuilder:AUDIOAMP_PAM8302A
- J4: device SparkFun-Connectors:CONN_02 -> SparkFun-Connectors:CONN_07
Connections:
- removed net N$26: R23.2, U7.IN_N
- removed net N$27: R24.2, U7.IN_P
- removed net N$28: C25.1, R23.1
- removed net N$29: FB4.P$1, U7.VO_N
- removed net N$30: FB3.P$1, U7.VO_P
- removed net N$31: C24.1, R24.1
- removed net N$32: C24.2, R26.1, R27.2
- removed net SD: R20.2, R25.2, U6./SD, U7./SD
- removed net VO+: C23.1, C28.1, FB1.P$2, FB3.P$2, J3.1, J4.1
- removed net VO-: C22.1, C27.1, FB2.P$2, FB4.P$2, J3.2, J4.2
- new net DTR: C29.1, J7.DTR
- new net N$13: C29.2, SJ2.2
- new net N$33: J7.RXI, R29.1
- new net N$34: J7.TXO, R30.1
- new net N$35: R31.2, U8.IN_N
- new net N$36: R32.2, U8.IN_P
- new net N$37: C33.1, R31.1
- new net N$38: FB6.P$1, U8.VO_N
- new net N$39: FB5.P$1, U8.VO_P
- new net N$40: C32.1, R32.1
- new net N$41: C32.2, C37.1, R34.1, R35.2
- new net SD1: R20.2, U6./SD
- new net SD2: R33.2, U8./SD
- new net VO1+: C23.1, FB1.P$2, J3.1
- new net VO1-: C22.1, FB2.P$2, J3.2
- new net VO2+: C36.1, FB5.P$2, J9.1
- new net VO2-: C35.1, FB6.P$2, J9.2
- net 3.3V: now also D4.C, R28.1
- net A1/0.03: now also J8.1
- net A2/0.04: now also J8.2
- net A3/0.05: now also J8.3
- net GND: now also C34.2, C35.2, C36.2, J7.GND, J8.4, U8.GND; no longer C26.2, C27.2, C28.2, U7.GND
- net N$25: now also C30.1
- net P0.07: now also C30.2
- net P0.15: now also R35.1; no longer R27.1
- net P0.16: now also C33.2, C37.2, R34.2; no longer C25.2, R26.2
- net RESET: now also D4.A, R28.2, SJ2.1
- net RXD: now also R30.2
- net TXD: now also R29.2
- net VBUS: now also J7.VCC
- net VCC_2: now also C34.1, R33.1, U8.VDD; no longer C26.1, R25.1, U7.VDD
Other:
- note added: "0.1uF+10K @ 3.3V = ~1.2ms to 0.7VCC"
- note added: "USB RESET (DTR)"

Commit message: update board
Parts:
- removed C32, C33: 1uF, microbuilder:CAP_CERAMIC0805-NOOUTLINE
- removed C34: 10uF, microbuilder:CAP_CERAMIC0805-NOOUTLINE
- removed R33: 10K, microbuilder:RESISTOR0805_NOOUTLINE
- added C24, C26: 1uF, rcl:C-EUC0805
- added C25: 10uF, rcl:C-EUC0805
- added R24: 10k, rcl:R-EU_R0805
- added SW3: SWITCH_SPDT, SparkFun-Retired:SWITCH_SPDT
- C1, C2: LCSC (none) -> C1836
- C10, C11, C14, C15, C16, C3, C5, C6, C8: LCSC (none) -> C1713
- C12: LCSC (none) -> C16005
- C13, C17, C18, C29: LCSC (none) -> C28378
- C19, C20: device microbuilder:CAP_CERAMIC0805-NOOUTLINE -> rcl:C-EUC0805; LCSC (none) -> C29822
- C21: device microbuilder:CAP_CERAMIC0805-NOOUTLINE -> rcl:C-EUC0805; LCSC (none) -> C1713
- C22, C23, C35, C36: LCSC (none) -> C46326
- C4: LCSC (none) -> C29822
- C7, C9: LCSC (none) -> C1735
- CHG: LCSC (none) -> C154481
- D1: LCSC (none) -> C72037
- D2: LCSC (none) -> C2293
- D4: LCSC (none) -> C99332
- D5: LCSC (none) -> C130880
- FB1, FB2, FB5, FB6: LCSC (none) -> C12389
- JP4: value SWO -> (none)
- L1, L2: LCSC (none) -> C112611
- Q3: LCSC (none) -> C10487
- R1, R13, R16, R2, R29, R3, R30: LCSC (none) -> C101404
- R10: LCSC (none) -> C101970
- R11, R12, R17, R5, R8, R9: LCSC (none) -> C103905
- R14, R15: LCSC (none) -> C101548
- R18, R19, R31, R32: LCSC (none) -> C153166
- R20: value 10K -> 10k; device microbuilder:RESISTOR0805_NOOUTLINE -> rcl:R-EU_R0805; LCSC (none) -> C84376
- R21, R22, R34, R35: LCSC (none) -> C84375
- R28, R7: LCSC (none) -> C84376
- R4: LCSC (none) -> C104516
- R6: LCSC (none) -> C26112
- U$45, U$51: DIGIKEY (none) -> 1568-1826-ND
- U1: DIGIKEY (none) -> 1597-1434-ND
- U2, U5: LCSC (none) -> C51118
- U3: LCSC (none) -> C14879
- U4: LCSC (none) -> C7974
- U6, U8: LCSC (none) -> C113367
- X2: DIGIKEY (none) -> 455-1749-1-ND
- X3: LCSC (none) -> C91146
- X4: LCSC (none) -> C48615
Connections:
- new net N$26: Q3.D, SW3.S
- net GND: now also C25.2; no longer C34.2
- net N$21: now also C20.2; no longer C20.1
- net N$24: now also C19.2; no longer C19.1
- net N$25: now also C19.1; no longer C19.2
- net N$37: now also C26.2; no longer C33.1
- net N$40: now also C24.2; no longer C32.1
- net N$41: now also C24.1; no longer C32.2
- net P0.07: now also C20.1; no longer C20.2
- net P0.16: now also C26.1; no longer C33.2
- net SD1: now also R20.1; no longer R20.2
- net SD2: now also R24.1; no longer R33.2
- net VBAT: now also SW3.P; no longer Q3.D
- net VCC_2: now also C25.1, R20.2, R24.2; no longer C34.1, R20.1, R33.1
Other:
- moved on the sheet: C19, C20, R20

Commit message: add fix
Other:
- note added: "ADD CLK PULLUP ON CLK OUT!"
- note added: "RXTX wrong!!!!"
Changed lines of the file:
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@@
 low Z at low F). Try to block everything
 &gt;1MHz or so.</text>
+<text x="-124.46" y="-25.4" size="6.4516" layer="95">RXTX wrong!!!!</text>
+<text x="45.72" y="-99.06" size="6.4516" layer="95">ADD CLK PULLUP ON CLK OUT!</text>
 </plain>
 <instances>
